File: temp-relay.kicad_sch (KiCad schematic)
At the start: 8 parts

Commit message: pcb update
Parts:
- C1: renamed from C?; footprint (none) -> Capacitor_THT:CP_Axial_L10.0mm_D4.5mm_P15.00mm_Horizontal
- R1, R2, R3: renamed from R?; footprint (none) -> Resistor_THT:R_Axial_DIN0204_L3.6mm_D1.6mm_P5.08mm_Horizontal
- SW1: renamed from SW?; footprint (none) -> Resistor_THT:R_Axial_DIN0204_L3.6mm_D1.6mm_P5.08mm_Horizontal
- gave numbers to parts that had none: 3
Connections:
- no-connect marks 0 -> 28
